Commit message: added readme

File: robot_config/niryo_ned2.urdf (robot description, URDF)
Before this commit: robot niryo_ned2, 10 links, 9 joints
Links:
- link arm_link: geometry collision mesh filename=package://niryo_ned_description/meshes/ned2/stl/arm_link.stl
- link base_link: geometry collision mesh filename=package://niryo_ned_description/meshes/ned2/stl/base_link.s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
- link elbow_link: geometry collision mesh filename=package://niryo_ned_description/meshes/ned2/stl/elbow_link.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
- link forearm_link: geometry collision mesh filename=package://niryo_ned_description/meshes/ned2/stl/forearm_lin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
- link hand_link: geometry collision mesh filename=package://niryo_ned_description/meshes/ned2/stl/hand_link.s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
- link shoulder_link: geometry collision mesh filename=package://niryo_ned_description/meshes/ned2/stl/shoulder_li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
- link wrist_link: geometry collision mesh filename=package://niryo_ned_description/meshes/ned2/stl/wrist_link.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
